Commit message: updated tracking, wbsite to view gui

File: tabletennistrainer_ws/src/ttt_control/urdf/mainarmass_fixed.urdf (robot description, URDF)
Before this commit: robot mainarmass, 7 links, 6 joints
Links:
- link Base: geometry collision mesh filename=package://ttt_control/meshes/67.stl scale=1 1 1; visual mesh filename=package://ttt_control/meshes/67.stl scale=1 1 1
- link Forearm: geometry collision mesh filename=package://ttt_control/meshes/79.stl scale=1 1 1; visual mesh filename=package://ttt_control/meshes/79.stl scale=1 1 1
- link Paddle: geometry collision mesh filename=package://ttt_control/meshes/71.stl scale=1 1 1; visual mesh filename=package://ttt_control/meshes/71.stl scale=1 1 1
- link Shoulder: geometry collision mesh filename=package://ttt_control/meshes/63.stl scale=1 1 1; visual mesh filename=package://ttt_control/meshes/63.stl scale=1 1 1
- link UpperArm: geometry collision mesh filename=package://ttt_control/meshes/75.stl scale=1 1 1; visual mesh filename=package://ttt_control/meshes/75.stl scale=1 1 1
- link Wrist: geometry collision mesh filename=package://ttt_control/meshes/59.stl scale=1 1 1; visual mesh filename=package://ttt_control/meshes/59.stl scale=1 1 1

Commit message: robot IK solver being worked on

File: tabletennistrainer_ws/src/ttt_control/urdf/mainarmass_fixed.urdf (robot description, URDF)
Before this commit: robot mainarmass, 7 links, 6 joints
Links:
- added link paddle_tcp; visual sphere radius=0.01
- added link table_surface; collision box size=2.0 2.0 0.02; visual box size=2.0 2.0 0.02
- link Forearm: mass 29.5338 -> 0.757
- link root: geometry visual sphere radius=0.001
Joints:
- added joint paddle_to_tcp: type fixed, parent Paddle, child paddle_tcp, origin xyz=-0.033 -0.105 0.149 rpy=-0.587 0.245 -1.933
- added joint table_to_base: type fixed, parent Base, child table_surface, origin xyz=0 0 0 rpy=0 0 0
- joint BaseRotate_0: limit effort=10.0 velocity=3.14 -> effort=35.0 velocity=5
- joint ForeArmRotate_0: limit effort=10.0 velocity=3.14 -> lower=-4.1888 upper=0.5236 effort=12.0 velocity=5; type continuous -> revolute
- joint PaddleRotate_0: limit effort=10.0 velocity=3.14 -> effort=0.75 velocity=5
- joint UpperArmRotate_0: limit effort=10.0 velocity=3.14 -> lower=-0.2617 upper=1.3963 effort=30.0 velocity=5; type continuous -> revolute
- joint WristRotate_0: limit effort=10.0 velocity=3.14 -> lower=-2.967 upper=2.50 effort=0.75 velocity=5; type continuous -> revolute

Commit message: urdf looks pretty nice

File: tabletennistrainer_ws/src/ttt_control/urdf/mainarmass_fixed.urdf (robot description, URDF)
Before this commit: robot mainarmass, 9 links, 8 joints
Links:
- added link table_center; visual sphere radius=0.05
- link table_surface: geometry collision box size=2.74 1.52 0.02; visual box size=2.74 1.52 0.02
Joints:
- removed joint table_to_base
- added joint center_to_robot: type fixed, parent table_center, child root, origin xyz=-1.37 0 0 rpy=0 0 3.14159
- added joint center_to_table: type fixed, parent table_center, child table_surface, origin xyz=0 0 0 rpy=0 0 0
- joint BaseRotate_0: axis 0.04806 -0.01710 -0.99869 -> 0.04806 -0.01710 0.99869

Commit message: this mayyyy be working

File: tabletennistrainer_ws/src/ttt_control/urdf/mainarmass_fixed.urdf (robot description, URDF)
Before this commit: robot mainarmass, 10 links, 9 joints
Joints:
- joint center_to_robot: origin xyz=-1.37 0 0 rpy=0 0 3.14159 -> xyz=-1.37 0 0 rpy=0 0 -1.5708

Commit message: im movin it

File: tabletennistrainer_ws/src/ttt_control/urdf/mainarmass_fixed.urdf (robot description, URDF)
Before this commit: robot mainarmass, 10 links, 9 joints
Joints:
- joint BaseRotate_0: limit effort=35.0 velocity=5 -> lower=-2.0944 upper=2.0944 effort=35.0 velocity=5; type continuous -> revolute
- joint ForeArmRotate_0: axis 0.93476 -0.35525 0 -> -0.93476 0.35525 0; limit lower=-4.1888 upper=0.5236 effort=12.0 velocity=5 -> lower=-0.436332 upper=2.6180 effort=12.0 velocity=5
- joint PaddleRotate_0: limit effort=0.75 velocity=5 -> lower=-1.5708 upper=1.5708 effort=0.75 velocity=5; type continuous -> revolute
- joint UpperArmRotate_0: limit lower=-0.2617 upper=1.3963 effort=30.0 velocity=5 -> lower=-0.261799 upper=1.0472 effort=30.0 velocity=5
- joint WristRotate_0: limit lower=-2.967 upper=0.2618 effort=0.75 velocity=5 -> lower=-1.5708 upper=1.5708 effort=0.75 velocity=5
- joint center_to_robot: origin xyz=-1.37 0 0 rpy=0 0 -1.5708 -> xyz=-1.37 0 0 rpy=0 0 0
- joint root_to_base: origin xyz=0 0 0 rpy=0 0 0 -> xyz=0 0 0 rpy=0 0 2.3736

Commit message: it hitta the ball

File: tabletennistrainer_ws/src/ttt_control/urdf/mainarmass_fixed.urdf (robot description, URDF)
Before this commit: robot mainarmass, 10 links, 9 joints
Joints:
- joint UpperArmRotate_0: limit lower=-0.261799 upper=1.0472 effort=30.0 velocity=5 -> lower=-0.261799 upper=0.5236 effort=30.0 velocity=5
- joint WristRotate_0: limit lower=-1.5708 upper=1.5708 effort=0.75 velocity=5 -> lower=2.0944 upper=3.14 effort=0.75 velocity=5

Commit message: wip on paddle and wrist urdf

File: tabletennistrainer_ws/src/ttt_control/urdf/mainarmass_fixed.urdf (robot description, URDF)
Before this commit: robot mainarmass, 10 links, 9 joints
Joints:
- joint WristRotate_0: limit lower=2.0944 upper=3.14 effort=0.75 velocity=5 -> lower=0.0 upper=3.14 effort=0.75 velocity=5

Commit message: shut up you chuds
I am god and I love windows

File: tabletennistrainer_ws/src/ttt_control/urdf/mainarmass_fixed.urdf (robot description, URDF)
Before this commit: robot mainarmass, 10 links, 9 joints
Joints:
- joint WristRotate_0: limit lower=0.0 upper=3.14 effort=0.75 velocity=5 -> lower=-3.14 upper=-1.57 effort=0.75 velocity=5

Commit message: i hate ik

File: tabletennistrainer_ws/src/ttt_control/urdf/mainarmass_fixed.urdf (robot description, URDF)
Before this commit: robot mainarmass, 10 links, 9 joints
Joints:
- joint ForeArmRotate_0: limit lower=-0.436332 upper=2.6180 effort=12.0 velocity=5 -> lower=-0.436332 upper=1.0472 effort=12.0 velocity=5
- joint WristRotate_0: limit lower=-3.14 upper=-1.57 effort=0.75 velocity=5 -> lower=-3.1415 upper=-1.5708 effort=0.75 velocity=5

Commit message: still wrist problems

File: tabletennistrainer_ws/src/ttt_control/urdf/mainarmass_fixed.urdf (robot description, URDF)
Before this commit: robot mainarmass, 10 links, 9 joints
Links:
- link paddle_tcp: geometry collision sphere radius=0.01; visual sphere radius=0.01
Joints:
- joint WristRotate_0: limit lower=-3.1415 upper=-1.5708 effort=0.75 velocity=5 -> lower=-3.1415 upper=3.14 effort=0.75 velocity=5

Commit message: docker container for moveit added, wrist and paddle joints are passive for now, need to update later

File: tabletennistrainer_ws/src/ttt_control/urdf/mainarmass_fixed.urdf (robot description, URDF)
Before this commit: robot mainarmass, 10 links, 9 joints
Joints:
- joint WristRotate_0: limit lower=-3.1415 upper=3.14 effort=0.75 velocity=5 -> lower=-3.14159 upper=0 effort=0.75 velocity=5; origin xyz=-0.10957 -0.19888 -0.43388 rpy=-0.84990 0.27810 3.0151 -> xyz=-0.10957 -0.19888 -0.43388 rpy=-2.48921 0.22754 2.49360

Commit message: ik works i thunk

File: tabletennistrainer_ws/src/ttt_control/urdf/mainarmass_fixed.urdf (robot description, URDF)
Before this commit: robot mainarmass, 10 links, 9 joints
Joints:
- joint ForeArmRotate_0: limit lower=-0.436332 upper=1.0472 effort=12.0 velocity=5 -> lower=-0.436332 upper=2.181 effort=12.0 velocity=5
- joint UpperArmRotate_0: limit lower=-0.261799 upper=0.5236 effort=30.0 velocity=5 -> lower=-0.261799 upper=2.705 effort=30.0 velocity=5

Commit message: reverted to z=0 tracking, limited base shoudler and arm joints, added STM command bottleneck

File: tabletennistrainer_ws/src/ttt_control/urdf/mainarmass_fixed.urdf (robot description, URDF)
Before this commit: robot mainarmass, 10 links, 9 joints
Joints:
- joint BaseRotate_0: limit lower=-2.0944 upper=2.0944 effort=35.0 velocity=5 -> lower=-0.959931 upper=0.959931 effort=35.0 velocity=5
- joint UpperArmRotate_0: limit lower=-0.261799 upper=2.705 effort=30.0 velocity=5 -> lower=-0.261799 upper=0.523599 effort=30.0 velocity=5

Commit message: urdf tweaks

File: tabletennistrainer_ws/src/ttt_control/urdf/mainarmass_fixed.urdf (robot description, URDF)
Before this commit: robot mainarmass, 10 links, 9 joints
Joints:
- joint BaseRotate_0: limit lower=-0.959931 upper=0.959931 effort=35.0 velocity=5 -> lower=-2.0944 upper=2.0944 effort=35.0 velocity=5
- joint ForeArmRotate_0: limit lower=-0.436332 upper=2.181 effort=12.0 velocity=5 -> lower=-0.436332 upper=1.0472 effort=12.0 velocity=5
- joint UpperArmRotate_0: limit lower=-0.261799 upper=0.523599 effort=30.0 velocity=5 -> lower=-0.261799 upper=0.5236 effort=30.0 velocity=5
